Commit message: Changes on inverted option of the angles, match simulation and leonardo robot on bicep and omoplate angles

File: inmoov_description/robots/inmoov.urdf.xacro (robot description, xacro)
@@ -90,5 +90,5 @@
    <axis xyz="1 0 0"/>
    <limit effort="1000.0" lower="${l_shoulder_out_joint_lower}" upper="${l_shoulder_out_joint_upper}" velocity="${l_shoulder_out_joint_velocity}" />
-   <origin rpy="0 0 0" xyz="0 0.143 0.298"/>
+   <origin rpy="-1.3963 0 0" xyz="0 0.143 0.298"/>
    <parent link="torso_link"/>
    <child link="l_shoulder_base_link"/>

File: inmoov_description/urdf/asmArm.urdf.xacro (robot description, xacro)
@@ -80,5 +80,5 @@
       <limit effort="1000.0" lower="${r_elbow_flex_joint_lower}" upper="${r_elbow_flex_joint_upper}" velocity="${r_elbow_flex_joint_velocity}" />
     </xacro:if>
-    <origin rpy="0 0 0" xyz="-0.0278 0 -0.2235"/>
+    <origin rpy="0 -1 0" xyz="-0.0278 0 -0.2235"/>
     <parent link="${side}_bicep_link"/>
     <child link="${side}_forearm_link"/>

Commit message: Changes on angles of right arm

File: inmoov_description/robots/inmoov.urdf.xacro (robot description, xacro)
@@ -72,7 +72,7 @@
   <xacro:arm side="r" flip="1" covers="yes" />
   <joint name="r_shoulder_out_joint" type="revolute">
-   <axis xyz="1 0 0"/>
+   <axis xyz="-1 0 0"/>
    <limit effort="1000.0" lower="${r_shoulder_out_joint_lower}" upper="${r_shoulder_out_joint_upper}" velocity="${r_shoulder_out_joint_velocity}" />
-   <origin rpy="0 0 0" xyz="0 -0.143 0.298"/>
+   <origin rpy="1.5708 0 0" xyz="0 -0.143 0.298"/>
    <parent link="torso_link"/>
    <child link="r_shoulder_base_link"/>

File: inmoov_description/urdf/asmArm.urdf.xacro (robot description, xacro)
@@ -52,21 +52,24 @@
     <xacro:if value="${side == 'l'}">
       <limit effort="1000.0" lower="${l_shoulder_lift_joint_lower}" upper="${l_shoulder_lift_joint_upper}" velocity="${l_shoulder_lift_joint_velocity}" />
+      <origin rpy="0 0.5236 0" xyz="0 ${flip * -0.012} -0.04"/>
     </xacro:if>
     <xacro:if value="${side == 'r'}">
       <limit effort="1000.0" lower="${r_shoulder_lift_joint_lower}" upper="${r_shoulder_lift_joint_upper}" velocity="${r_shoulder_lift_joint_velocity}" />
+      <origin rpy="0 0 0" xyz="0 ${flip * -0.012} -0.04"/>
     </xacro:if>
-    <origin rpy="0 0.5236 0" xyz="0 ${flip * -0.012} -0.04"/>
     <parent link="${side}_shoulder_base_link"/>
     <child link="${side}_shoulder_link"/>
   </joint>
   <joint name="${side}_upper_arm_roll_joint" type="revolute">
-    <axis xyz="0 0 1"/>
     <xacro:if value="${side == 'l'}">
+      <axis xyz="0 0 1"/>
       <limit effort="1000.0" lower="${l_upper_arm_roll_joint_lower}" upper="${l_upper_arm_roll_joint_upper}" velocity="${l_upper_arm_roll_joint_velocity}" />
+      <origin rpy="0 0 -1.5708" xyz="0 ${flip * -0.066} -0.060"/>
     </xacro:if>
     <xacro:if value="${side == 'r'}">
+      <axis xyz="0 0 -1"/>
       <limit effort="1000.0" lower="${r_upper_arm_roll_joint_lower}" upper="${r_upper_arm_roll_joint_upper}" velocity="${r_upper_arm_roll_joint_velocity}" />
+      <origin rpy="0 0 0.959549361" xyz="0 ${flip * -0.066} -0.060"/>
     </xacro:if>
-    <origin rpy="0 0 -1.5708" xyz="0 ${flip * -0.066} -0.060"/>
     <parent link="${side}_shoulder_link"/>
     <child link="${side}_bicep_link"/>
@@ -78,5 +81,5 @@
     </xacro:if>
     <xacro:if value="${side == 'r'}">
-      <axis xyz="0 1 0"/>
+      <axis xyz="0 -1 0"/>
       <limit effort="1000.0" lower="${r_elbow_flex_joint_lower}" upper="${r_elbow_flex_joint_upper}" velocity="${r_elbow_flex_joint_velocity}" />
     </xacro:if>

Commit message: Rotate hands

File: inmoov_description/robots/inmoov.urdf.xacro (robot description, xacro)
@@ -82,5 +82,5 @@
    <axis xyz="0 0 1"/>
    <limit effort="1000.0" lower="${r_wrist_roll_joint_lower}" upper="${r_wrist_roll_joint_upper}" velocity="${r_wrist_roll_joint_velocity}" />
-   <origin rpy="0 0 0" xyz="-0.0144 0.01  -0.2885"/>
+   <origin rpy="0 0 -3.1416" xyz="-0.0144 0.01  -0.2885"/>
    <parent link="r_forearm_link"/>
    <child link="r_hand_link"/>
@@ -98,5 +98,5 @@
    <axis xyz="0 0 1"/>
    <limit effort="1000.0" lower="${l_wrist_roll_joint_lower}" upper="${l_wrist_roll_joint_upper}" velocity="${l_wrist_roll_joint_velocity}" />
-   <origin rpy="0 0 0" xyz="-0.0144 -0.01  -0.2885"/>
+   <origin rpy="0 0 3.1416" xyz="-0.0144 -0.01  -0.2885"/>
    <parent link="l_forearm_link"/>
    <child link="l_hand_link"/>

Commit message: Change angles of head to match with physical leonardo GreenMoov

File: inmoov_description/robots/inmoov.urdf.xacro (robot description, xacro)
@@ -59,5 +59,5 @@
    <axis xyz="0 1 0"/>
    <limit effort="1000.0" lower="${head_tilt_joint_lower}" upper="${head_tilt_joint_upper}" velocity="${head_tilt_joint_velocity}" />
-   <origin rpy="0 0 3.1415" xyz="0 0 0"/>
+   <origin rpy="0 -1.0472 3.1415" xyz="0 0 0"/>
    <parent link="head_tilt_link"/>
    <child link="head_base_link"/>

File: inmoov_description/urdf/asmHead.urdf.xacro (robot description, xacro)
@@ -61,5 +61,5 @@
    <axis xyz="0 0 1"/>
    <limit effort="1000.0" lower="${head_pan_joint_lower}" upper="${head_pan_joint_upper}" velocity="${head_pan_joint_velocity}" />
-   <origin rpy="0 0 0" xyz="0 0 0.0245"/>
+   <origin rpy="0 0 -0.8726" xyz="0 0 0.0245"/>
    <parent link="head_base_link"/>
    <child link="head_link"/>

Commit message: Corrections on the angles o the head

File: inmoov_description/robots/inmoov.urdf.xacro (robot description, xacro)
@@ -57,7 +57,8 @@
   </joint>
   <joint name="head_tilt_joint" type="revolute">
-   <axis xyz="0 1 0"/>
+   <axis xyz="0 -1 0"/>
    <limit effort="1000.0" lower="${head_tilt_joint_lower}" upper="${head_tilt_joint_upper}" velocity="${head_tilt_joint_velocity}" />
-   <origin rpy="0 -1.0472 3.1415" xyz="0 0 0"/>
+   <!-- <origin rpy="0 -1.0472 3.1415" xyz="0 0 0"/> -->
+   <origin rpy="0 -5.236 3.1415" xyz="0 0 0"/>
    <parent link="head_tilt_link"/>
    <child link="head_base_link"/>

File: inmoov_description/urdf/asmHead.urdf.xacro (robot description, xacro)
@@ -61,5 +61,5 @@
    <axis xyz="0 0 1"/>
    <limit effort="1000.0" lower="${head_pan_joint_lower}" upper="${head_pan_joint_upper}" velocity="${head_pan_joint_velocity}" />
-   <origin rpy="0 0 -0.8726" xyz="0 0 0.0245"/>
+   <origin rpy="0 0 -1.7453" xyz="0 0 0.0245"/>
    <parent link="head_base_link"/>
    <child link="head_link"/>
