Commit message: Changes Angles of shoulder for leonardo

File: inmoov_description/urdf/asmArm.urdf.xacro (robot description, xacro)
@@ -49,5 +49,5 @@
   </link>
   <joint name="${side}_shoulder_lift_joint" type="revolute">
-    <axis xyz="0 1 0"/>
+    <axis xyz="0 -1 0"/>
     <xacro:if value="${side == 'l'}">
       <limit effort="1000.0" lower="${l_shoulder_lift_joint_lower}" upper="${l_shoulder_lift_joint_upper}" velocity="${l_shoulder_lift_joint_velocity}" />
@@ -56,5 +56,5 @@
       <limit effort="1000.0" lower="${r_shoulder_lift_joint_lower}" upper="${r_shoulder_lift_joint_upper}" velocity="${r_shoulder_lift_joint_velocity}" />
     </xacro:if>
-    <origin rpy="0 0 0" xyz="0 ${flip * -0.012} -0.04"/>
+    <origin rpy="0 0.5236 0" xyz="0 ${flip * -0.012} -0.04"/>
     <parent link="${side}_shoulder_base_link"/>
     <child link="${side}_shoulder_link"/>

Commit message: Change angles of rotate of left arm of leonardo

File: inmoov_description/urdf/asmArm.urdf.xacro (robot description, xacro)
@@ -68,5 +68,5 @@
       <limit effort="1000.0" lower="${r_upper_arm_roll_joint_lower}" upper="${r_upper_arm_roll_joint_upper}" velocity="${r_upper_arm_roll_joint_velocity}" />
     </xacro:if>
-    <origin rpy="0 0 0" xyz="0 ${flip * -0.066} -0.060"/>
+    <origin rpy="0 0 -1.5708" xyz="0 ${flip * -0.066} -0.060"/>
     <parent link="${side}_shoulder_link"/>
     <child link="${side}_bicep_link"/>

Commit message: Fix on the inversed angle control, disabled some nodes on launchfile that are not used, and fix on the bicep of the virtual inmoov

File: inmoov_description/urdf/asmArm.urdf.xacro (robot description, xacro)
@@ -73,12 +73,13 @@
   </joint>
   <joint name="${side}_elbow_flex_joint" type="revolute">
-    <axis xyz="0 1 0"/>
     <xacro:if value="${side == 'l'}">
+      <axis xyz="0 -1 0"/>
       <limit effort="1000.0" lower="${l_elbow_flex_joint_lower}" upper="${l_elbow_flex_joint_upper}" velocity="${l_elbow_flex_joint_velocity}" />
     </xacro:if>
     <xacro:if value="${side == 'r'}">
+      <axis xyz="0 1 0"/>
       <limit effort="1000.0" lower="${r_elbow_flex_joint_lower}" upper="${r_elbow_flex_joint_upper}" velocity="${r_elbow_flex_joint_velocity}" />
     </xacro:if>
-    <origin rpy="0 -1 0" xyz="-0.0278 0 -0.2235"/>
+    <origin rpy="0 0 0" xyz="-0.0278 0 -0.2235"/>
     <parent link="${side}_bicep_link"/>
     <child link="${side}_forearm_link"/>

Commit message: perception listener

File: inmoov_description/urdf/asmArm.urdf.xacro (robot description, xacro)
@@ -71,4 +71,5 @@
       <limit effort="1000.0" lower="${r_upper_arm_roll_joint_lower}" upper="${r_upper_arm_roll_joint_upper}" velocity="${r_upper_arm_roll_joint_velocity}" />
       <origin rpy="0 0 0.959549361" xyz="0 ${flip * -0.066} -0.060"/>
+      <!-- <origin rpy="0 0 0.959549361" xyz="0 -0.066 -0.060"/> -->
     </xacro:if>
     <parent link="${side}_shoulder_link"/>
